File: HW/Test Circuits/Motor Measurement/mm.kicad_pcb (KiCad board)
At the start: 2 copper layers, 22 parts, among them J1 IN, J2 MOTOR, J3 PWR, J4 OUT, U1 MCP6002

Commit message: The first wave of test boards finished
Parts:
- moved C1 138.6 mm to (245.1, 28.6)
- moved C3 138.6 mm to (251.5, 29.2)
- moved D1 138.6 mm to (241.9, 52.7)
- moved HEATSINK_TO220 138.6 mm to (238.1, 52.7)
- moved J1 138.6 mm to (228.0, 45.7)
- moved R1 138.6 mm to (229.9, 55.2)
- moved R10 138.6 mm to (253.4, 62.9)
- moved R8 138.6 mm to (245.7, 52.1)
- moved U1 138.6 mm to (252.1, 50.8)
- moved C2 138.6 mm to (258.4, 36.8)
- moved C4 138.6 mm to (258.4, 50.8)
- moved DP5050 138.6 mm to (242.6, 46.4)
- moved J2 138.6 mm to (233.0, 27.3)
- moved J3 138.6 mm to (262.9, 47.0)
- moved J4 138.6 mm to (262.9, 56.5)
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Other:
- board outline added: 50 x 50 mm
