File: HW/Test Circuits/P-Channel Driver/pcd.sch (KiCad schematic (older format))
At the start: 15 parts, among them J1 PWR, J2 PWM_IN, J3 OUT, Q1 BC546B, Q2 BC546B, Q3 IRF9530

Commit message: The first wave of test boards finished
Parts:
- J1: footprint CONN_NCW254-02S -> MOLEX_36538_2
Connections:
- net GND: now also J1.1 (P1); no longer J1.2 (PM)
- net VDD: now also J1.2 (PM); no longer J1.1 (P1), R1.1
- net at D2.2 (K), F1.2, Q3.3 (S)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: now also R1.1
Changed lines of the file:
@@
 LIBS:contrib
 LIBS:valves
+LIBS:pcd-cache
 EELAYER 27 0
 EELAYER END
@@
 Sheet 1 1
 Title ""
-Date "12 feb 2015"
+Date "13 feb 2015"
 Rev ""
 Comp ""
@@
 Wire Wire Line
 	3150 3275 3150 3300
-$Comp
-L VDD #PWR03
-U 1 1 54C359A3
-P 2325 2975
-F 0 "#PWR03" H 2325 3075 30  0001 C CNN
-F 1 "VDD" H 2325 3085 30  0000 C CNN
-F 2 "" H 2325 2975 60  0000 C CNN
-F 3 "" H 2325 2975 60  0000 C CNN
-	1    2325 2975
-	-1   0    0    -1
-$EndComp
 Wire Wire Line
 	2325 2975 2325 3050
@@
 F 0 "J1" V 1600 3450 40  0000 C CNN
 F 1 "PWR" V 1700 3450 40  0000 C CNN
-F 2 "CONN_NCW254-02S" H 1650 3450 60  0001 C CNN
+F 2 "MOLEX_36538_2" H 1650 3450 60  0001 C CNN
 F 3 "" H 1650 3450 60  0000 C CNN
 	1    1650 3450
-	-1   0    0    -1
+	-1   0    0    1
 $EndComp
 $Comp
@@
 	4350 4075 4350 4300
 $Comp
-L GND #PWR04
+L GND #PWR03
 U 1 1 54DCABA5
 P 4350 4800
-F 0 "#PWR04" H 4350 4800 30  0001 C CNN
+F 0 "#PWR03" H 4350 4800 30  0001 C CNN
 F 1 "GND" H 4350 4730 30  0001 C CNN
 F 2 "" H 4350 4800 60  0000 C CNN
@@
 	4350 4700 4350 4800
 $Comp
-L GND #PWR05
+L GND #PWR04
 U 1 1 54DCABCD
 P 2000 4850
-F 0 "#PWR05" H 2000 4850 30  0001 C CNN
+F 0 "#PWR04" H 2000 4850 30  0001 C CNN
 F 1 "GND" H 2000 4780 30  0001 C CNN
 F 2 "" H 2000 4850 60  0000 C CNN
@@
 	2000 4725 2000 4850
 $Comp
-L GND #PWR06
+L GND #PWR05
 U 1 1 54DCABF6
 P 2000 3650
-F 0 "#PWR06" H 2000 3650 30  0001 C CNN
+F 0 "#PWR05" H 2000 3650 30  0001 C CNN
 F 1 "GND" H 2000 3580 30  0001 C CNN
 F 2 "" H 2000 3650 60  0000 C CNN
@@
 	2000 3550 2000 3650
 $Comp
-L VDD #PWR07
+L VDD #PWR06
 U 1 1 54DCAC20
 P 2000 3275
-F 0 "#PWR07" H 2000 3375 30  0001 C CNN
+F 0 "#PWR06" H 2000 3375 30  0001 C CNN
 F 1 "VDD" H 2000 3385 30  0000 C CNN
 F 2 "" H 2000 3275 60  0000 C CNN
@@
 	2000 3275 2000 3350
 $Comp
-L GND #PWR08
+L GND #PWR07
 U 1 1 54DCAC4B
 P 5100 4800
-F 0 "#PWR08" H 5100 4800 30  0001 C CNN
+F 0 "#PWR07" H 5100 4800 30  0001 C CNN
 F 1 "GND" H 5100 4730 30  0001 C CNN
 F 2 "" H 5100 4800 60  0000 C CNN
@@
 Connection ~ 5100 4700
 Connection ~ 4800 4000
+Wire Wire Line
+	2325 2975 3800 2975
+Wire Wire Line
+	3800 2975 3800 3275
 $EndSCHEMATC

Commit message: Updated MOSFET driver circuit/simulation added
Parts:
- D1: value DIODESCH -> 1N5819
- D2: value ZENER -> BZX85C10
Changed lines of the file:
@@
 Sheet 1 1
 Title ""
-Date "13 feb 2015"
+Date "18 apr 2015"
 Rev ""
 Comp ""
@@
 P 3800 3475
 F 0 "D2" H 3800 3575 50  0000 C CNN
-F 1 "ZENER" H 3800 3375 40  0000 C CNN
+F 1 "BZX85C10" H 3800 3375 40  0000 C CNN
 F 2 "D2" H 3800 3475 60  0001 C CNN
 F 3 "" H 3800 3475 60  0000 C CNN
@@
 P 2575 3500
 F 0 "D1" H 2575 3600 40  0000 C CNN
-F 1 "DIODESCH" H 2575 3400 40  0000 C CNN
+F 1 "1N5819" H 2575 3400 40  0000 C CNN
 F 2 "D2" H 2575 3500 60  0001 C CNN
 F 3 "" H 2575 3500 60  0000 C CNN
