File: HW/Test Circuits/Driver V1/driver.sch (KiCad schematic (older format))
At the start: 23 parts

Commit message: Driver schematic (unfinished)
Parts:
- removed C? (x3): 10uF/63V, ~, symbol C
- removed C?: 1000uF/63V, ~, symbol CP
- removed C?: 1000uF/63V, C3P_D7, symbol CP
- removed C?: 10nF/100V, C2, symbol C
- removed D?: ZENER, D2, symbol ZENER
- removed D?: DIODESCH, D2, symbol DIODESCH
- removed D?: MBR10100, TO220-2, symbol DIODE-HEXFRED
- removed F?: FUSE, AUTOFUSE, symbol FUSE
- removed J?: OUT, MD-TEST-HDR-M, symbol MD-TEST-HDR
- removed J?: PWR, MOLEX_36538_2, symbol CONN_2
- removed J?: PWM_IN, CONN_NCW254-02S, symbol CONN_2
- removed L?: INDUCTOR, ~, symbol INDUCTOR
- removed L?: 470uH/10A, L-TOROID-D35X5, symbol INDUCTOR
- removed Q?: IRF9530, TO-220_V, symbol MOSFET_P_GDS
- removed Q? (x2): BC546B, TO-92_V, symbol NPN_CBE
- removed R? (x2): 750/2W, R6, symbol R
- removed R?: 1K8, R4, symbol R
- removed R?: 1, R4, symbol R
- removed R?: 100, R4, symbol R
- added C1: 100uF/63V, ~, symbol CP
- added C10: 1uF/63V, C2_3x1,75, symbol C
- added C11, C12: 10nF, C2, symbol C
- added C13: 100nF, C1, symbol C
- added C2, C4, C7: 10uF/63V, ~, symbol C
- added C3: 470nF/100V, ~, symbol C
- added C5: 1000uF/63V, ~, symbol CP
- added C6: 220uF/10V, C1P_D2.7, symbol CP
- added C8: 1000uF/63V, C3P_D7, symbol CP
- added C9: 10nF/100V, C2, symbol C
- added D1: 1N5817, D4, symbol DIODESCH
- added D2: DIODESCH, D2, symbol DIODESCH
- added D3: BZX55C10, D2, symbol ZENER
- added D4, D5: MBR10100, TO220-2, symbol DIODE-HEXFRED
- added F1: FUSE, AUTOFUSE, symbol FUSE
- added J1: PWR, MOLEX_36538_2, symbol CONN_2
- added J2: PWM_IN, CONN_NCW254-02S, symbol CONN_2
- added J3: MOTOR, MOLEX_36538_2, symbol CONN_2
- added J4: OUT, CONN_NCW254-04S, symbol CONN_4
- added L1: 10uH/500mA, ~, symbol INDUCTOR
- added L2: 10uH/10A, ~, symbol INDUCTOR
- added L3: 100uH, R5, symbol INDUCTOR
- added L4: 470uH/10A, L-TOROID-D35X5, symbol INDUCTOR
- added Q1, Q2: BC546B, TO-92_V, symbol NPN_CBE
- added Q3: IRF9530, TO-220_V, symbol MOSFET_P_GDS
- added R1: 100, R4, symbol R
- added R10, R11, R12: 10K, R4, symbol R
- added R13: 100K, R4, symbol R
- added R14: 680K, R4, symbol R
- added R15: 390K, R4, symbol R
- added R2, R5: 750/2W, R6, symbol R
- added R3: 1, R4, symbol R
- added R4: 1K8, R4, symbol R
- added R6: R005/1W, R4_5_6, symbol R
- added R7: 1K, R4, symbol R
- added R8, R9: 220K, R4, symbol R
- added U1: LM2594HVM-5.0, DIP-8, symbol LM2594
- added U2: MCP6002, DIP-8, symbol MCP6002
Connections:
- net GND: now also C1.2, C12.2, C13.2, C2.2, C3.2, C4.2, C5.2, C6.2, C7.2, C8.2, C9.2, D1.1 (A), D4.3 (A), J1.1 (P1), J2.2 (PM), J4.4 (P4), Q2.3 (E), R10.1, R12.2, R6.2, R9.2, U1.5 (~ON~/OFF), U1.6 (GND), U2.4 (V-), U2.4 (V-)
- net VDD: now also C2.1, C4.1, F1.2, L1.1, L2.1
- new net: F1.1, J1.2 (PM)
- new net: D3.1 (A), Q1.3 (E), Q3.1 (G), R5.2
- new net: D4.1 (K), L4.1, Q3.2 (D)
- new net: C5.1, C7.1, D3.2 (K), L2.2, Q3.3 (S), R1.1, R3.1
- new net: Q2.1 (C), R2.1, R5.1
- new net: Q2.2 (B), R4.1
- new net: J2.1 (P1), R4.2
- new net: Q1.1 (C), R3.2
- new net: D2.2 (K), Q1.2 (B)
- new net: D2.1 (A), R1.2, R2.2
- new net: C8.1, C9.1, J3.2 (PM), L4.2
- new net: D5.1 (K), R6.1, U2.5 (+)
- new net: C10.1, D5.3 (A), J3.1 (P1)
- new net: C10.2, R7.1
- new net: C11.2, C12.1, R7.2, R8.2, R9.1, U2.2 (-)
- new net: R11.2, R12.1, R14.1, U2.3 (+)
- new net: J4.2 (P2), R14.2, U2.1
- new net: R10.2, R13.1, U2.6 (-)
- new net: J4.1 (P1), R15.2, U2.7
- new net: R13.2, R15.1
- new net: C1.1, C3.1, L1.2, U1.7 (IN)
- new net: D1.2 (K), L3.1, U1.8 (OUT)
- new net VCC: C11.1, C13.1, C6.1, J4.3 (P3), L3.2, R11.1, R8.1, U1.4 (FB), U2.8 (V+), U2.8 (V+)
