File: HW/Test Circuits/Driver V1/driver.sch (KiCad schematic (older format))
At the start: 47 parts, among them J1 PWR, J2 PWM_IN, J3 MOTOR, J4 OUT, Q1 BC546B, Q2 BC546B, Q3 IRF9530, U1 LM2594HVM-5.0, U2 MCP6002

Commit message: Protection diodes added to the schematic, changed to 3.3V
Parts:
- added D? (x2): MBR10100, TO220-2, symbol DIODE-HEXFRED
- U1: value LM2594HVM-5.0 -> LM2594HVM-3.3
Connections:
- net at C8.1, C9.1, J3.2 (PM)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: now also D?.1 (K)
- net at C10.1, D5.3 (A), J3.1 (P1): now also D?.3 (A)
- new net: D?.1 (K), D?.3 (A)
Other:
- moved on the sheet: C11, C12, C13, J4, R10, R11, R12, R13, R14, R15, R7, R8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
