File: HW/Test Circuits/Logic PSU/PSU.sch (KiCad schematic (older format))
At the start: 15 parts

Commit message: Logic PSU Test board updated +cleaning
Parts:
- removed C? (x2): CP, ~, symbol CP
- removed C?: 470pF, ~, symbol C
- removed D?: DIODESCH, ~, symbol DIODESCH
- removed D? (x2): 33V, ~, symbol ZENER-SOT23
- removed D?: 15V, ~, symbol ZENER-SOT23
- removed L?: INDUCTOR, ~, symbol INDUCTOR
- removed Q?: MOSFET_P_GDS, ~, symbol MOSFET_P_GDS
- removed R? (x5): R, ~, symbol R
- removed U?: MC34063, ~, symbol MC34063
- added C1: 100uF/63V, Capacitors_SMD:c_elec_10x10.5, symbol CP
- added C2: 220uF/10V Tantalum, Capacitors_Tantalum_SMD:TantalC_SizeD_EIA-7343_HandSoldering, symbol CP
- added C3: 100uF/6.3V Tantalum, Capacitors_Tantalum_SMD:TantalC_SizeB_EIA-3528_HandSoldering, symbol CP
- added D1: SS14, Diodes_SMD:Diode-SMA_Handsoldering, symbol DIODESCH
- added J1: PWR, suf_connector_ncw:CONN_NCW396-02R, symbol CONN_2
- added J2: OUT, suf_connector_ncw:CONN_NCW396-02R, symbol CONN_2
- added L1: 100uH, Choke_SMD:Choke_SMD_Wuerth-WE-PD-Typ-LS_Handsoldering, symbol INDUCTOR
- added L2: 3.3uH, Choke_SMD:Choke_SMD_Wuerth-WE-PD-Typ-M-Typ-S_Handsoldering, symbol INDUCTOR
- added U1: LM2594HVM-3.3, Housings_SOIC:SOIC-8_3.9x4.9mm_Pitch1.27mm, symbol LM2594
Connections:
- net labels added: VDD
- net labels removed: VEE
- wire segments 34 -> 19
