File: HW/Test Circuits/MCU Board v1/MCU.sch (KiCad schematic (older format))
At the start: 15 parts

Commit message: MCU Board v1 updated +cleanup DO NOT BUILD IT, BUGGY !!!
Parts:
- removed C?: 1uF TANTAL, ~, symbol CP
- removed C? (x2): 100n, ~, symbol C
- removed C?: 10uF/10V TANTAL, ~, symbol CP
- removed C? (x2): C, ~, symbol C
- removed L? (x2): INDUCTOR, ~, symbol INDUCTOR
- removed P? (x2): CONN_24, symbol CONN_24
- removed R? (x2): R, ~, symbol R
- removed X?: XTAL, ~, symbol XTAL
- added C1, C2: 10nF, Capacitors_ThroughHole:C_Rect_L4_W2.5_P2.5, symbol C
- added E1: EC11P20, suf_switch:EC11P20_single_side, symbol EC11P20
- added J2: MODE, suf_connector_ncw:CONN_NCW254-03S, symbol CONN_3
- added J3: I2C, suf_connector_ncw:CONN_NCW254-03S, symbol CONN_3
- added J4: PWM, suf_connector_ncw:CONN_NCW254-03S, symbol CONN_3
- added J5: CAL, suf_connector_ncw:CONN_NCW254-02S, symbol CONN_2
- added J6: PWM_DUAL, Pin_Headers:Pin_Header_Straight_1x03, symbol CONN_3
- added J7: PWM_IN, suf_connector_ncw:CONN_NCW254-02S, symbol CONN_2
- added R1, R3, R6, R7, R8, R9: 10K, Resistors_ThroughHole:Resistor_Horizontal_RM10mm, symbol R
- added R10: 3R9, Resistors_ThroughHole:Resistor_Horizontal_RM10mm, symbol R
- added R2, R4, R5: 47K, Resistors_ThroughHole:Resistor_Horizontal_RM10mm, symbol R
- added U1: CONRAD_USB_UART, suf_module:CONRAD_USB_UART, symbol CONRAD_USB_UART
- added U3: TJCTM24028-SPI, suf_display:TJCTM24028-SPI, symbol TJCTM24028-SPI
- J1: renamed from P?; value CONN_5 -> Measure; footprint (none) -> suf_connector_ncw:CONN_NCW254-05S
- U2: renamed from U?; value M054LDN -> M0516LDN; footprint ~ -> suf_module:M0516-DEV
Connections:
- net labels added: ADC_I, ADC_U, CAL, ENC_A, ENC_B, I2C_SCL, I2C_SDA, MODE_AUTO, MODE_RPM, PWM_0, PWM_1, RPM_CTRL, RPM_IN, RXD, TFT_CS, TFT_DC, TFT_MISO, TFT_MOSI, TFT_RST, TFT_SCK, TXD
- net labels removed: AGND, VDD
- wire segments 154 -> 99
Other:
- moved on the sheet: J1, U2
