File: HW/Test Circuits/Motor Measurement v2/mm.sch (KiCad schematic (older format))
At the start: 47 parts, among them J1 IN, J2 MOTOR, J3 PWR, J4 OUT, J5 CONN_9X2, U1 MCP6002, U2 MCP6002

Commit message: Motor Measurement v2 cleanup
Parts:
- D1, D2: value MBR10100 -> MBR10200
- R10, R11, R12, R13, R14, R15, R16, R17, R18, R19, R2, R20, R21, R22, R3, R4, R5, R6, R7, R9: footprint R4 -> Discret:R4
- R8: value 21K -> 1K1; footprint R4 -> Discret:R4
Other:
- moved on the sheet: C1, C10, C11, C12, C13, C2, C3, C4, C5, C6, C7, C8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
